File: NatSi-DevKit/NatSi-DevKit.kicad_sch (KiCad schematic)
At the start: 52 parts, among them J1 USB_TypeC, J2 Conn_01x22_Pin, J3 Conn_01x22_Pin, J4 MEM2067-02-180-00-A_REVB, SW1 SW_Push, SW2 SW_Push, SW3 SW_Push, U1 USBLC6-2SC6, U2 ESP32-S3-WROOM-1, U3 NCP1117-3.3_SOT223

Commit message: ooooh its done :3
Parts:
- added TP15: TestPoint, sumec_graphic:UWU_IMG, symbol Connector:TestPoint
- TP5: renamed from TP7; footprint sumec_graphic:BLAHAJ_LINE_IMG -> sumec_graphic:BLAHAJ_SOLDER_LN_IMG
- TP7: renamed from TP9; footprint sumec_graphic:JOJO_SYMBOL_IMG -> sumec_graphic:JOJO_SOLDER_IMG
- renumbered TP12 to TP10, TP13 to TP11, TP14 to TP12, TP15 to TP13, TP16 to TP14, TP4 to TP3, TP5 to TP4, TP8 to TP6, TP10 to TP8, TP11 to TP9
Connections:
- net JOJO renamed JOJO_SOLDER
- new net UWU: TP15.1
Changed lines of the file:
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@@
 	(wire
 		(pts
+			(xy 360.68 229.87) (xy 360.68 215.9)
+		)
+		(stroke
+			(width 0)
+			(type default)
+		)
+	)
+	(wire
+		(pts
 			(xy 341.63 229.87) (xy 341.63 215.9)
 		)
@@
 		)
 	)
-	(label "JOJO"
+	(label "JOJO_SOLDER"
 		(at 330.2 229.87 90)
 		(fields_autoplaced yes)
@@
 		)
 	)
+	(label "UWU"
+		(at 360.68 229.87 90)
+		(fields_autoplaced yes)
+		(effects
+			(font
+				(size 1.27 1.27)
+			)
+			(justify left bottom)
+		)
+	)
 	(label "NYA~"
 		(at 356.87 229.87 90)
@@
 		(on_board yes)
 		(dnp no)
-		(property "Reference" "TP13"
+		(property "Reference" "TP11"
 			(at 347.218 211.328 0)
 			(effects
@@
 			(project "NatSi-DevKit"
 				(path "/900bd7ac-cdf9-4a2f-8b1f-2c21e3760046"
-					(reference "TP13")
+					(reference "TP11")
 					(unit 1)
 				)
@@
 		(on_board yes)
 		(dnp no)
-		(property "Reference" "TP11"
+		(property "Reference" "TP9"
 			(at 339.598 211.328 0)
 			(effects
@@
 			(project "NatSi-DevKit"
 				(path "/900bd7ac-cdf9-4a2f-8b1f-2c21e3760046"
-					(reference "TP11")
+					(reference "TP9")
 					(unit 1)
 				)
@@
 		(on_board yes)
 		(dnp no)
-		(property "Reference" "TP4"
+		(property "Reference" "TP3"
 			(at 316.738 211.328 0)
 			(effects
@@
 			(project "NatSi-DevKit"
 				(path "/900bd7ac-cdf9-4a2f-8b1f-2c21e3760046"
-					(reference "TP4")
+					(reference "TP3")
 					(unit 1)
 				)
@@
 		(on_board yes)
 		(dnp no)
-		(property "Reference" "TP5"
+		(property "Reference" "TP4"
 			(at 320.548 211.328 0)
 			(effects
@@
 			(project "NatSi-DevKit"
 				(path "/900bd7ac-cdf9-4a2f-8b1f-2c21e3760046"
-					(reference "TP5")
+					(reference "TP4")
 					(unit 1)
 				)
@@
 		(on_board yes)
 		(dnp no)
-		(property "Reference" "TP14"
+		(property "Reference" "TP12"
 			(at 351.028 211.328 0)
 			(effects
@@
 			(project "NatSi-DevKit"
 				(path "/900bd7ac-cdf9-4a2f-8b1f-2c21e3760046"
-					(reference "TP14")
+					(reference "TP12")
 					(unit 1)
 				)
@@
 		(on_board yes)
 		(dnp no)
-		(property "Reference" "TP7"
+		(property "Reference" "TP5"
 			(at 324.358 211.328 0)
 			(effects
@@
 			)
 		)
-		(property "Footprint" "sumec_graphic:BLAHAJ_LINE_IMG"
+		(property "Footprint" "sumec_graphic:BLAHAJ_SOLDER_LN_IMG"
 			(at 327.66 222.885 0)
 			(effects
@@
 			(project "NatSi-DevKit"
 				(path "/900bd7ac-cdf9-4a2f-8b1f-2c21e3760046"
-					(reference "TP7")
+					(reference "TP5")
 					(unit 1)
 				)
@@
 	)
 	(symbol
+		(lib_id "Connector:TestPoint")
+		(at 360.68 215.9 0)
+		(unit 1)
+		(exclude_from_sim no)
+		(in_bom yes)
+		(on_board yes)
+		(dnp no)
+		(property "Reference" "TP15"
+			(at 362.458 211.328 0)
+			(effects
+				(font
+					(face "Consolas")
+					(size 1.27 1.27)
+				)
+				(justify left)
+				(hide yes)
+			)
+		)
+		(property "Value" "TestPoint"
+			(at 362.458 213.868 0)
+			(effects
+				(font
+					(face "Consolas")
+					(size 1.27 1.27)
+				)
+				(justify left)
+				(hide yes)
+			)
+		)
+		(property "Footprint" "sumec_graphic:UWU_IMG"
+			(at 365.76 222.885 0)
+			(effects
+				(font
+					(face "Consolas")
+					(size 1.27 1.27)
+				)
+				(hide yes)
+			)
+		)
+		(property "Datasheet" "~"
+			(at 365.76 215.9 0)
+			(effects
+				(font
+					(face "Consolas")
+					(size 1.27 1.27)
+				)
+				(hide yes)
+			)
+		)
+		(property "Description" "test point"
+			(at 360.68 215.9 0)
+			(effects
+				(font
+					(face "Consolas")
+					(size 1.27 1.27)
+				)
+				(hide yes)
+			)
+		)
+		(pin "1"
+		)
+		(instances
+			(project "NatSi-DevKit"
+				(path "/900bd7ac-cdf9-4a2f-8b1f-2c21e3760046"
+					(reference "TP15")
+					(unit 1)
+				)
+			)
+		)
+	)
+	(symbol
 		(lib_id "power:GND")
 		(at 109.22 184.15 0)
@@
 		(on_board yes)
 		(dnp no)
-		(property "Reference" "TP10"
+		(property "Reference" "TP8"
 			(at 335.788 211.328 0)
 			(effects
@@
 			(project "NatSi-DevKit"
 				(path "/900bd7ac-cdf9-4a2f-8b1f-2c21e3760046"
-					(reference "TP10")
+					(reference "TP8")
 					(unit 1)
 				)
@@
 		(on_board yes)
 		(dnp no)
-		(property "Reference" "TP8"
+		(property "Reference" "TP6"
 			(at 328.168 211.328 0)
 			(effects
@@
 			(project "NatSi-DevKit"
 				(path "/900bd7ac-cdf9-4a2f-8b1f-2c21e3760046"
-					(reference "TP8")
+					(reference "TP6")
 					(unit 1)
 				)
@@
 		(on_board yes)
 		(dnp no)
-		(property "Reference" "TP15"
+		(property "Reference" "TP13"
 			(at 354.838 211.328 0)
 			(effects
@@
 			(project "NatSi-DevKit"
 				(path "/900bd7ac-cdf9-4a2f-8b1f-2c21e3760046"
-					(reference "TP15")
+					(reference "TP13")
 					(unit 1)
 				)
@@
 		(on_board yes)
 		(dnp no)
-		(property "Reference" "TP9"
+		(property "Reference" "TP7"
 			(at 331.978 211.328 0)
 			(effects
@@
 			)
 		)
-		(property "Footprint" "sumec_graphic:JOJO_SYMBOL_IMG"
+		(property "Footprint" "sumec_graphic:JOJO_SOLDER_IMG"
 			(at 335.28 222.885 0)
 			(effects
@@
 			(project "NatSi-DevKit"
 				(path "/900bd7ac-cdf9-4a2f-8b1f-2c21e3760046"
-					(reference "TP9")
+					(reference "TP7")
 					(unit 1)
 				)
@@
 		(on_board yes)
 		(dnp no)
-		(property "Reference" "TP16"
+		(property "Reference" "TP14"
 			(at 358.648 211.328 0)
 			(effects
@@
 			(project "NatSi-DevKit"
 				(path "/900bd7ac-cdf9-4a2f-8b1f-2c21e3760046"
-					(reference "TP16")
+					(reference "TP14")
 					(unit 1)
 				)
@@
 		(on_board yes)
 		(dnp no)
-		(property "Reference" "TP12"
+		(property "Reference" "TP10"
 			(at 343.408 211.328 0)
 			(effects
@@
 			(project "NatSi-DevKit"
 				(path "/900bd7ac-cdf9-4a2f-8b1f-2c21e3760046"
-					(reference "TP12")
+					(reference "TP10")
 					(unit 1)
 				)
