File: NatSi-DevKit/NatSi-DevKit.kicad_pcb (KiCad board)
At the start: 4 copper layers, 62.5 x 25.4 mm, 60 parts, among them J1 USB_TypeC, J2 Conn_01x22_Pin, J3 Conn_01x22_Pin, J4 MEM2067-02-180-00-A_REVB, SW1 SW_Push, SW2 SW_Push, SW3 SW_Push, U1 USBLC6-2SC6, U2 ESP32-S3-WROOM-1, U3 NCP1117-3.3_SOT223

Commit message: ooooh its done :3
Parts:
- removed the TP9 at (113.7, 110.6)
- removed the TP9 at (115.5, 107.5)
- added TP13: TestPoint, sumec_graphic:OWO_IMG, F.Cu at (167.2, 97.5)
- added TP15: TestPoint, sumec_graphic:UWU_IMG, F.Cu at (171.4, 103.3)
- added TP7: TestPoint, sumec_graphic:JOJO_SOLDER_IMG, B.Cu at (113.4, 110.5)
- added TP9: TestPoint, sumec_graphic:JOJO_SOLDER_IMG, B.Cu at (115.2, 107.3)
- TP5: renamed from TP7; footprint sumec_graphic:BLAHAJ_LINE_IMG -> sumec_graphic:BLAHAJ_SOLDER_LN_IMG
- moved TP11 11.0 mm to (170.7, 107.3), turned to 135 degrees
- moved TP8 10.4 mm to (165.8, 98.4), turned to 90 degrees
- moved TP5 10.0 mm to (143.7, 97.9)
- moved TP3 1.37 mm to (114.7, 100.9)
- renumbered TP12 to TP10, TP13 to TP11, TP14 to TP12, TP16 to TP14, TP4 to TP3, TP5 to TP4, TP8 to TP6, TP10 to TP8, TP11 to TP9

Commit message: you will get your present soon cutie :3
Other:
- board text added: "STRAPPING PINS: D0,D3,D45,D46 ADC1: D1-D10 ADC2: D11-D20 USB: D19-, D20+"
- board text removed: "STRAPPING PINS:D0,D3,D45,D46 ADC1:D1-D10, ADC2:D11-D20"

Commit message: not sure whats the diff
Other:
- board text added: "text"
Changed lines of the file:
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@@
 		(layer "F.Fab")
+	)
+	(gr_text "text"
+		(at 183.215 130.03 0)
+		(layer "B.Cu" knockout)
+		(effects
+			(font
+				(size 1.5 1.5)
+				(thickness 0.3)
+				(bold yes)
+			)
+			(justify left bottom mirror)
+		)
 	)
 	(gr_text "D02"

Commit message: some minor changes
Other:
- board text removed: "text"
Changed lines of the file:
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@@
 		(layer "Edge.Cuts")
 	)
-	(gr_line
-		(start 219.30673 48.64687)
-		(end 222.7844 45.1692)
-		(stroke
-			(width 0.2)
-			(type default)
-		)
-		(layer "F.Fab")
-	)
-	(gr_line
-		(start 234.664431 48.667231)
-		(end 231.165284 45.168084)
-		(stroke
-			(width 0.2)
-			(type default)
-		)
-		(layer "F.Fab")
-	)
-	(gr_line
-		(start 221.9716 45.9312)
-		(end 232.5888 45.9312)
-		(stroke
-			(width 0.1)
-			(type default)
-		)
-		(layer "F.Fab")
-	)
-	(gr_text "text"
-		(at 183.215 130.03 0)
-		(layer "B.Cu" knockout)
-		(effects
-			(font
-				(size 1.5 1.5)
-				(thickness 0.3)
-				(bold yes)
-			)
-			(justify left bottom mirror)
-		)
-	)
 	(gr_text "5V"
 		(at 122.683 89.797 0)
@@
 				)
 			)
-		)
-	)
-	(dimension
-		(type aligned)
-		(layer "F.Fab")
-		(pts
-			(xy 236.7544 45.9312) (xy 231.9792 45.9312)
-		)
-		(height 2.9972)
-		(format
-			(prefix "")
-			(suffix "")
-			(units 3)
-			(units_format 1)
-			(precision 4)
-		)
-		(style
-			(thickness 0.1)
-			(arrow_length 1.27)
-			(text_position_mode 0)
-			(arrow_direction outward)
-			(extension_height 0.58642)
-			(extension_offset 0.5)
-			(keep_text_aligned yes)
-		)
-		(gr_text "4.7752 mm"
-			(at 234.3668 41.784 0)
-			(layer "F.Fab")
-			(effects
-				(font
-					(size 1 1)
-					(thickness 0.15)
-				)
-			)
